File: hardware/schematics/van-obc/Sensors.kicad_sch (KiCad schematic)
At the start: 5 parts, among them J5 J_BME, J6 J_MPU, J7 J_MQ2, J8 J_MQ7, J9 J_DS18B20

Commit message: fix(tests): Corrections majeures KY040, BME280, MPU6050
- KY040 v2.1.0: Fix comptage + anti-rebond capacitif
- BME280 v1.0.1: Fix begin() avec &Wire
- MPU6050 v2.0.0: Simplification (acc only, dérive <2°)
- Ajout diagnostic_bme280.ino + CHANGELOG

Tests: 6/11 validés (55%)
Parts:
- J5, J6: footprint (none) -> Connector_PinHeader_2.54mm:PinHeader_1x04_P2.54mm_Vertical
- J7, J8, J9: footprint (none) -> Connector_PinHeader_2.54mm:PinHeader_1x03_P2.54mm_Vertical
Changed lines of the file:
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@@
 	(title_block
 		(title "Van Onboard Computer")
-		(date "2025-11-30")
-		(rev "1.0")
+		(date "2025-12-02")
+		(rev "1.1")
 	)
 	(text "+5V"
@@
 			)
 		)
-		(property "Footprint" ""
+		(property "Footprint" "Connector_PinHeader_2.54mm:PinHeader_1x04_P2.54mm_Vertical"
 			(at 63.5 40.64 0)
 			(effects
@@
 			)
 		)
-		(property "Footprint" ""
+		(property "Footprint" "Connector_PinHeader_2.54mm:PinHeader_1x04_P2.54mm_Vertical"
 			(at 63.5 59.69 0)
 			(effects
@@
 			)
 		)
-		(property "Footprint" ""
+		(property "Footprint" "Connector_PinHeader_2.54mm:PinHeader_1x03_P2.54mm_Vertical"
 			(at 63.5 113.03 0)
 			(effects
@@
 			)
 		)
-		(property "Footprint" ""
+		(property "Footprint" "Connector_PinHeader_2.54mm:PinHeader_1x03_P2.54mm_Vertical"
 			(at 63.5 96.52 0)
 			(effects
@@
 			)
 		)
-		(property "Footprint" ""
+		(property "Footprint" "Connector_PinHeader_2.54mm:PinHeader_1x03_P2.54mm_Vertical"
 			(at 63.5 80.01 0)
 			(effects
